Commit message: Adding new mount locations for 3d print

File: urdf/magni.urdf.xacro (robot description, xacro)
@@ -82,5 +82,7 @@
     <parent link="base_footprint"/>
     <child link="rplidar"/>
-    <origin xyz="-0.047 0 0.3" rpy="0 0 0"/>
+    <!-- <origin xyz="-0.047 0 0.3" rpy="0 0 0"/> -->
+    <!-- moved in x by 2cm up in z by 2.5cm -->
+    <origin xyz="-0.027 0 0.325" rpy="0 0 0"/>
   </joint>
   <!-- Macro for defining wheels -->
@@ -176,5 +178,7 @@
     <xacro:if value="${raspicam_mount == 'upward'}">
       <xacro:raspi_camera name="raspicam" connected_to="base_link">
-        <origin xyz="0.020 0.115 0.155" rpy="0 0 ${pi}"/>
+        <!-- <origin xyz="0.020 0.115 0.155" rpy="0 0 ${pi}"/> -->
+        <!-- new camera mount is roughly deltas of x=+0.01 y=-0.01 z=+0.02   -->
+        <origin xyz="0.03 0.105 0.175" rpi="0 0 ${pi}" />
       </xacro:raspi_camera>
     </xacro:if>

Commit message: attempting to rotate the camera in xarco

File: urdf/magni.urdf.xacro (robot description, xacro)
@@ -180,5 +180,5 @@
         <!-- <origin xyz="0.020 0.115 0.155" rpy="0 0 ${pi}"/> -->
         <!-- new camera mount is roughly deltas of x=+0.01 y=-0.01 z=+0.02   -->
-        <origin xyz="0.03 0.105 0.175" rpi="0 0 ${pi}" />
+        <origin xyz="0.03 0.105 0.175" rpy="0 0 0" />
       </xacro:raspi_camera>
     </xacro:if>

Commit message: Attempting calibration again

File: urdf/magni.urdf.xacro (robot description, xacro)
@@ -180,5 +180,5 @@
         <!-- <origin xyz="0.020 0.115 0.155" rpy="0 0 ${pi}"/> -->
         <!-- new camera mount is roughly deltas of x=+0.01 y=-0.01 z=+0.02   -->
-        <origin xyz="0.03 0.105 0.175" rpy="0 0 0" />
+        <origin xyz="0.03 0.105 0.175" rpy="0 0 1.57070" />
       </xacro:raspi_camera>
     </xacro:if>

Commit message: updated sensor placement

File: urdf/magni.urdf.xacro (robot description, xacro)
@@ -156,41 +156,10 @@
   </xacro:if>
   <!-- If we are given an extrinsics calibration use that instead of the pre-configured pose -->
-  <xacro:if value="${camera_extrinsics_file != '-'}">
-    <xacro:property name="cam_extrinsics" value="${load_yaml(camera_extrinsics_file)}"/>
-    <xacro:property name="cam_position" value="${cam_extrinsics['position']}"/>
-    <xacro:property name="cam_orientation" value="${cam_extrinsics['orientation']}"/>
-    <xacro:raspi_camera name="raspicam" connected_to="base_link">
-      <origin xyz="${cam_position['x']} ${cam_position['y']} ${cam_position['z']}"
-        rpy="${cam_orientation['r']} ${cam_orientation['p']} ${cam_orientation['y']}"/>
-    </xacro:raspi_camera>
-  </xacro:if>
-  <xacro:if value="${camera_extrinsics_file == '-'}">
     <!-- Define raspicam based on the raspicam_mount argument -->
-    <!-- forward  Forward and tilted slightly upwards         -->
     <!-- upward   Pointing straight up                        -->
-    <!-- downward High on post and pointing 45 degree down    -->
-    <!-- ahead    Directly facing forward with no tilt        -->
-    <xacro:if value="${raspicam_mount == 'forward'}">
-      <xacro:raspi_camera name="raspicam" connected_to="base_link">
-        <origin xyz="0.050 0.085 0.135" rpy="1.15191731 0 1.5707"/>
-      </xacro:raspi_camera>
-    </xacro:if>
-    <xacro:if value="${raspicam_mount == 'upward'}">
       <xacro:raspi_camera name="raspicam" connected_to="base_link">
         <!-- <origin xyz="0.020 0.115 0.155" rpy="0 0 ${pi}"/> -->
         <!-- new camera mount is roughly deltas of x=+0.01 y=-0.01 z=+0.02   -->
-        <origin xyz="0.03 0.105 0.175" rpy="0 0 1.57070" />
+        <origin xyz="0.03 0.105 0.175" rpy="0 0 -${pi/2}" />
       </xacro:raspi_camera>
-    </xacro:if>
-    <xacro:if value="${raspicam_mount == 'downward'}">
-      <xacro:raspi_camera name="raspicam" connected_to="base_link">
-        <origin xyz="0.1 0.090 0.145" rpy="3.14159 -1.25 0.0"/>
-      </xacro:raspi_camera>
-    </xacro:if>
-    <xacro:if value="${raspicam_mount == 'ahead'}">
-      <xacro:raspi_camera name="raspicam" connected_to="base_link">
-        <origin xyz="0.095 0.061 0.10" rpy="0 1.5707 0"/>
-      </xacro:raspi_camera>
-    </xacro:if>
-  </xacro:if>
 </robot>

Commit message: first pass at new calibration params

File: urdf/magni.urdf.xacro (robot description, xacro)
@@ -84,5 +84,6 @@
     <!-- <origin xyz="-0.047 0 0.3" rpy="0 0 0"/> -->
     <!-- moved in x by 2cm up in z by 2.5cm -->
-    <origin xyz="-0.027 0 0.325" rpy="0 0 0"/>
+    <!-- 3d print <origin xyz="-0.027 0 0.325" rpy="0 0 0"/> -->
+    <origin xyz="-0.93 0 0.198" rpy="0 0 0"/>
   </joint>
   <!-- Macro for defining wheels -->
@@ -161,5 +162,5 @@
         <!-- <origin xyz="0.020 0.115 0.155" rpy="0 0 ${pi}"/> -->
         <!-- new camera mount is roughly deltas of x=+0.01 y=-0.01 z=+0.02   -->
-        <origin xyz="0.03 0.105 0.175" rpy="0 0 -${pi/2}" />
+        <origin xyz="0.122 -0.03 1.06" rpy="0 0 ${pi/2}" />
       </xacro:raspi_camera>
 </robot>
